File: placa/GASOMETRO.kicad_pcb (KiCad board)
At the start: 2 copper layers, 19 parts, among them J1 USB_B, J2 Buzzer, J3 MQ5, J4 MQ7, J5 BMP180, J6 TEMT6000, J7 DatosOled, J8 AlimentacionOled, U1 LM317L_TO92, U2 ESP32-Devkit-V1

Commit message: fdgdf
Parts:
- moved U1 7.92 mm to (208.5, 114.6)
- moved R5 2.95 mm to (232.6, 110.4)
- moved R6 2.95 mm to (217.4, 114.6)
Routing:
- net +3V3: track 235.3 -> 246.0 mm
- net Net-(R5-Pad2): track 8.15 -> 13.1 mm
Changed lines of the file:
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@@
   )
   (footprint "Package_TO_SOT_THT:TO-92_Inline" (layer "F.Cu")
-    (at 216.4588 114.6004 180)
+    (at 208.534 114.6004 180)
     (descr "TO-92 leads in-line, narrow, oval pads, drill 0.75mm (see NXP sot054_po.pdf)")
     (tags "to-92 sc-43 sc-43a sot54 PA33 transistor")
@@
   )
   (footprint "Resistor_THT:R_Axial_DIN0309_L9.0mm_D3.2mm_P15.24mm_Horizontal" (layer "F.Cu")
-    (at 235.5596 110.3884 180)
+    (at 232.6132 110.3884 180)
     (descr "Resistor, Axial_DIN0309 series, Axial, Horizontal, pin pitch=15.24mm, 0.5W = 1/2W, length*diameter=9*3.2mm^2, http://cdn-reichelt.de/documents/datenblatt/B400/1_4W%23YAG.pdf")
     (tags "Resistor Axial_DIN0309 series Axial Horizontal pin pitch 15.24mm 0.5W = 1/2W length 9mm diameter 3.2mm")
@@
   )
   (footprint "Resistor_THT:R_Axial_DIN0309_L9.0mm_D3.2mm_P15.24mm_Horizontal" (layer "F.Cu")
-    (at 220.3704 114.6048)
+    (at 217.424 114.6048)
     (descr "Resistor, Axial_DIN0309 series, Axial, Horizontal, pin pitch=15.24mm, 0.5W = 1/2W, length*diameter=9*3.2mm^2, http://cdn-reichelt.de/documents/datenblatt/B400/1_4W%23YAG.pdf")
     (tags "Resistor Axial_DIN0309 series Axial Horizontal pin pitch 15.24mm 0.5W = 1/2W length 9mm diameter 3.2mm")
@@
   )
   (gr_rect (start 162.56 30.1244) (end 262.56 130.1244) (layer "B.Cu") (width 0.2) (fill none))
-  (segment (start 220.3196 110.3884) (end 220.3196 114.554) (width 1) (layer "B.Cu") (net 1))
-  (segment (start 216.4632 114.6048) (end 216.4588 114.6004) (width 1) (layer "B.Cu") (net 1))
-  (segment (start 220.3196 114.554) (end 220.3704 114.6048) (width 1) (layer "B.Cu") (net 1))
-  (segment (start 220.3704 114.6048) (end 216.4632 114.6048) (width 1) (layer "B.Cu") (net 1))
+  (segment (start 217.3732 110.3884) (end 217.3732 114.554) (width 1) (layer "B.Cu") (net 1))
+  (segment (start 217.3732 114.554) (end 217.424 114.6048) (width 1) (layer "B.Cu") (net 1))
+  (segment (start 217.424 114.6048) (end 208.5384 114.6048) (width 1) (layer "B.Cu") (net 1))
+  (segment (start 208.5384 114.6048) (end 208.534 114.6004) (width 1) (layer "B.Cu") (net 1))
   (segment (start 238.506 59.3344) (end 242.1128 59.3344) (width 1) (layer "F.Cu") (net 2))
   (via (at 242.1128 59.3344) (size 0.8) (drill 0.4) (layers "F.Cu" "B.Cu") (net 2))
@@
   (segment (start 188.5088 81.8488) (end 189.992 80.3656) (width 1) (layer "B.Cu") (net 2))
   (segment (start 235.641277 102.534323) (end 239.014 102.534323) (width 1) (layer "B.Cu") (net 2))
-  (segment (start 215.1888 114.6004) (end 215.1888 102.534323) (width 1) (layer "B.Cu") (net 2))
   (segment (start 189.992 53.6448) (end 190.5508 53.086) (width 1) (layer "B.Cu") (net 2))
   (segment (start 235.5596 102.452646) (end 235.641277 102.534323) (width 1) (layer "B.Cu") (net 2))
   (segment (start 242.1128 59.3344) (end 242.1128 102.362) (width 1) (layer "B.Cu") (net 2))
+  (segment (start 207.599677 102.534323) (end 215.1888 102.534323) (width 1) (layer "B.Cu") (net 2))
   (segment (start 235.5596 92.451) (end 235.5596 102.452646) (width 1) (layer "B.Cu") (net 2))
   (segment (start 172.974 81.8488) (end 188.5088 81.8488) (width 1) (layer "B.Cu") (net 2))
@@
   (segment (start 239.0648 102.585123) (end 239.014 102.534323) (width 1) (layer "B.Cu") (net 2))
   (segment (start 238.4552 59.2836) (end 238.506 59.3344) (width 1) (layer "B.Cu") (net 2))
+  (segment (start 207.264 102.87) (end 207.599677 102.534323) (width 1) (layer "B.Cu") (net 2))
   (segment (start 235.5596 102.616) (end 235.641277 102.534323) (width 1) (layer "B.Cu") (net 2))
   (segment (start 251.3076 102.585123) (end 241.889677 102.585123) (width 1) (layer "B.Cu") (net 2))
+  (segment (start 235.5596 110.3884) (end 232.6132 110.3884) (width 1) (layer "B.Cu") (net 2))
+  (segment (start 207.264 114.6004) (end 207.264 102.87) (width 1) (layer "B.Cu") (net 2))
   (segment (start 241.889677 102.585123) (end 239.0648 102.585123) (width 1) (layer "B.Cu") (net 2))
   (segment (start 189.992 80.3656) (end 189.992 53.6448) (width 1) (layer "B.Cu") (net 2))
@@
   (via (at 198.882 102.9716) (size 0.8) (drill 0.4) (layers "F.Cu" "B.Cu") (net 3))
   (via (at 192.3288 102.9716) (size 0.8) (drill 0.4) (layers "F.Cu" "B.Cu") (net 3))
+  (segment (start 205.994 118.11) (end 205.994 114.6004) (width 1) (layer "B.Cu") (net 3))
   (segment (start 213.848 121.5401) (end 240.4099 121.5401) (width 1) (layer "B.Cu") (net 3))
+  (segment (start 213.848 121.5401) (end 213.848 118.13) (width 1) (layer "B.Cu") (net 3))
   (segment (start 198.9215 102.9321) (end 198.9215 102.8079) (width 1) (layer "B.Cu") (net 3))
+  (segment (start 213.848 118.13) (end 213.868 118.11) (width 1) (layer "B.Cu") (net 3))
   (segment (start 165.1 63.2968) (end 165.1 102.9716) (width 1) (layer "B.Cu") (net 3))
   (segment (start 240.4099 121.5401) (end 242.691523 119.258477) (width 1) (layer "B.Cu") (net 3))
-  (segment (start 213.848 121.5401) (end 213.848 114.6712) (width 1) (layer "B.Cu") (net 3))
+  (segment (start 213.868 118.11) (end 205.994 118.11) (width 1) (layer "B.Cu") (net 3))
   (segment (start 172.6184 63.2968) (end 172.6184 68.082) (width 1) (layer "B.Cu") (net 3))
   (segment (start 198.9215 102.8079) (end 198.9215 92.2782) (width 1) (layer "B.Cu") (net 3))
+  (segment (start 205.994 114.6004) (end 198.9792 114.6004) (width 1) (layer "B.Cu") (net 3))
   (segment (start 198.9215 114.5427) (end 198.9215 102.8079) (width 1) (layer "B.Cu") (net 3))
   (segment (start 198.9792 114.6004) (end 198.9215 114.5427) (width 1) (layer "B.Cu") (net 3))
-  (segment (start 213.9188 114.6004) (end 198.9792 114.6004) (width 1) (layer "B.Cu") (net 3))
-  (segment (start 213.848 114.6712) (end 213.9188 114.6004) (width 1) (layer "B.Cu") (net 3))
   (segment (start 172.6184 63.2968) (end 165.1 63.2968) (width 1) (layer "B.Cu") (net 3))
   (segment (start 165.1 102.9716) (end 192.3288 102.9716) (width 1) (layer "B.Cu") (net 3))
